Commit message: feat: PS4 controller integration - software 90% complete, physical motion pending

File: src/aero_description/urdf/aero.ignition.xacro (robot description, xacro)
@@ -40,6 +40,10 @@
     </gazebo>
     <gazebo>
-        <plugin filename="libgz_ros2_control-system.so" name="gz_ros2_control::GazeboSimROS2ControlPlugin">
+        <plugin filename="ign_ros2_control-system" name="ign_ros2_control::IgnitionROS2ControlPlugin">
             <parameters>/home/ali/Desktop/Ros2_Control/install/aero_bringup/share/aero_bringup/config/controllers.yaml</parameters>
+            <ros>
+                <namespace></namespace>
+                <remapping>/controller_manager/robot_description:=/robot_description</remapping>
+            </ros>
         </plugin>
         <plugin filename="libignition-gazebo-imu-system.so"
@@ -52,3 +56,36 @@
         </plugin>
     </gazebo>
+    <!-- Wheel friction properties for Ignition Gazebo -->
+    <gazebo reference="front_right_wheel_link">
+        <mu1>2.0</mu1>
+        <mu2>2.0</mu2>
+        <kp>10000000.0</kp>
+        <kd>1.0</kd>
+        <minDepth>0.005</minDepth>
+        <fdir1>1 0 0</fdir1>
+    </gazebo>
+    <gazebo reference="front_left_wheel_link">
+        <mu1>2.0</mu1>
+        <mu2>2.0</mu2>
+        <kp>10000000.0</kp>
+        <kd>1.0</kd>
+        <minDepth>0.005</minDepth>
+        <fdir1>1 0 0</fdir1>
+    </gazebo>
+    <gazebo reference="back_right_wheel_link">
+        <mu1>2.0</mu1>
+        <mu2>2.0</mu2>
+        <kp>10000000.0</kp>
+        <kd>1.0</kd>
+        <minDepth>0.005</minDepth>
+        <fdir1>1 0 0</fdir1>
+    </gazebo>
+    <gazebo reference="back_left_wheel_link">
+        <mu1>2.0</mu1>
+        <mu2>2.0</mu2>
+        <kp>10000000.0</kp>
+        <kd>1.0</kd>
+        <minDepth>0.005</minDepth>
+        <fdir1>1 0 0</fdir1>
+    </gazebo>
 </robot>

File: src/aero_description/urdf/mobile_base.ros2_control.xacro (robot description, xacro)
@@ -2,20 +2,42 @@
 <robot xmlns:xacro="http://www.ros.org/wiki/xacro">
     <xacro:if value="${use_ignition}">
-        <ros2_control name="GazeboSimSystem" type="system">
+        <ros2_control name="IgnitionSystem" type="system">
             <hardware>
-                <plugin>gz_ros2_control/GazeboSimSystem</plugin>
+                <plugin>ign_ros2_control/IgnitionSystem</plugin>
+                <param name="robot_param">robot_description</param>
+                <param name="robot_param_node">robot_state_publisher</param>
             </hardware>
-            <xacro:macro name="gazebo_joint" params="name">
-                <joint name="${name}">
-                    <command_interface name="velocity" />
-                    <command_interface name="position" />
-                    <state_interface name="position" />
-                    <state_interface name="velocity"/>
-                </joint>
-            </xacro:macro>
-            <xacro:gazebo_joint name="base_front_right_wheel_joint" />
-            <xacro:gazebo_joint name="base_front_left_wheel_joint" />
-            <xacro:gazebo_joint name="base_back_right_wheel_joint" />
-            <xacro:gazebo_joint name="base_back_left_wheel_joint" />
+            <joint name="base_front_right_wheel_joint">
+                <command_interface name="velocity">
+                    <param name="min">-10</param>
+                    <param name="max">10</param>
+                </command_interface>
+                <state_interface name="position"/>
+                <state_interface name="velocity"/>
+            </joint>
+            <joint name="base_front_left_wheel_joint">
+                <command_interface name="velocity">
+                    <param name="min">-10</param>
+                    <param name="max">10</param>
+                </command_interface>
+                <state_interface name="position"/>
+                <state_interface name="velocity"/>
+            </joint>
+            <joint name="base_back_right_wheel_joint">
+                <command_interface name="velocity">
+                    <param name="min">-10</param>
+                    <param name="max">10</param>
+                </command_interface>
+                <state_interface name="position"/>
+                <state_interface name="velocity"/>
+            </joint>
+            <joint name="base_back_left_wheel_joint">
+                <command_interface name="velocity">
+                    <param name="min">-10</param>
+                    <param name="max">10</param>
+                </command_interface>
+                <state_interface name="position"/>
+                <state_interface name="velocity"/>
+            </joint>
         </ros2_control>
     </xacro:if>

Commit message: error no ros2 control tag

File: src/aero_description/urdf/aero.ignition.xacro (robot description, xacro)
@@ -40,6 +40,8 @@
     </gazebo>
     <gazebo>
-        <plugin filename="ign_ros2_control-system" name="ign_ros2_control::IgnitionROS2ControlPlugin">
+        <plugin filename="gz_ros2_control-system" name="gz_ros2_control::GazeboSimROS2ControlPlugin">
             <parameters>/home/ali/Desktop/Ros2_Control/install/aero_bringup/share/aero_bringup/config/controllers.yaml</parameters>
+            <robot_param>robot_description</robot_param>
+            <robot_param_node>robot_state_publisher</robot_param_node>
             <ros>
                 <namespace></namespace>

File: src/aero_description/urdf/mobile_base.ros2_control.xacro (robot description, xacro)
@@ -2,7 +2,7 @@
 <robot xmlns:xacro="http://www.ros.org/wiki/xacro">
     <xacro:if value="${use_ignition}">
-        <ros2_control name="IgnitionSystem" type="system">
+        <ros2_control name="GazeboSystem" type="system">
             <hardware>
-                <plugin>ign_ros2_control/IgnitionSystem</plugin>
+                <plugin>gz_ros2_control/GazeboSimSystem</plugin>
                 <param name="robot_param">robot_description</param>
                 <param name="robot_param_node">robot_state_publisher</param>
@@ -40,4 +40,37 @@
                 <state_interface name="velocity"/>
             </joint>
+            <!-- ARM JOINTS -->
+            <joint name="arm_joint0">
+                <command_interface name="position">
+                    <param name="min">-6.28</param>
+                    <param name="max">6.28</param>
+                </command_interface>
+                <state_interface name="position"/>
+                <state_interface name="velocity"/>
+            </joint>
+            <joint name="arm_joint1">
+                <command_interface name="position">
+                    <param name="min">-6.28</param>
+                    <param name="max">6.28</param>
+                </command_interface>
+                <state_interface name="position"/>
+                <state_interface name="velocity"/>
+            </joint>
+            <joint name="arm_joint2">
+                <command_interface name="position">
+                    <param name="min">-6.28</param>
+                    <param name="max">6.28</param>
+                </command_interface>
+                <state_interface name="position"/>
+                <state_interface name="velocity"/>
+            </joint>
+            <joint name="arm_joint3">
+                <command_interface name="position">
+                    <param name="min">-6.28</param>
+                    <param name="max">6.28</param>
+                </command_interface>
+                <state_interface name="position"/>
+                <state_interface name="velocity"/>
+            </joint>
         </ros2_control>
     </xacro:if>
