Commit message: The driving was interrupted, there's a mistake.

File: src/aero_description/urdf/aero.gazebo.xacro (robot description, xacro)
@@ -1,4 +1,102 @@
 <?xml version="1.0"?>
 <robot xmlns:xacro="http://www.ros.org/wiki/xacro">
-    <gazebo></gazebo>
+    <!-- Gazebo Classic ros2_control plugin -->
+    <gazebo>
+        <plugin filename="libgazebo_ros2_control.so" name="gazebo_ros2_control">
+            <robot_param>robot_description</robot_param>
+            <robot_param_node>robot_state_publisher</robot_param_node>
+            <parameters>$(find aero_bringup)/config/controllers.yaml</parameters>
+        </plugin>
+    </gazebo>
+    <!-- Gazebo Classic ros2_control hardware interface -->
+    <ros2_control name="GazeboSystem" type="system">
+        <hardware>
+            <plugin>gazebo_ros2_control/GazeboSystem</plugin>
+        </hardware>
+        <!-- Wheel joints -->
+        <joint name="base_front_left_wheel_joint">
+            <command_interface name="velocity">
+                <param name="min">-10</param>
+                <param name="max">10</param>
+            </command_interface>
+            <state_interface name="position"/>
+            <state_interface name="velocity"/>
+        </joint>
+        <joint name="base_front_right_wheel_joint">
+            <command_interface name="velocity">
+                <param name="min">-10</param>
+                <param name="max">10</param>
+            </command_interface>
+            <state_interface name="position"/>
+            <state_interface name="velocity"/>
+        </joint>
+        <joint name="base_back_left_wheel_joint">
+            <command_interface name="velocity">
+                <param name="min">-10</param>
+                <param name="max">10</param>
+            </command_interface>
+            <state_interface name="position"/>
+            <state_interface name="velocity"/>
+        </joint>
+        <joint name="base_back_right_wheel_joint">
+            <command_interface name="velocity">
+                <param name="min">-10</param>
+                <param name="max">10</param>
+            </command_interface>
+            <state_interface name="position"/>
+            <state_interface name="velocity"/>
+        </joint>
+        <!-- Arm joints -->
+        <xacro:if value="$(arg arm_enabled)">
+            <joint name="$(arg arm_prefix)joint0">
+                <command_interface name="position"/>
+                <state_interface name="position"/>
+                <state_interface name="velocity"/>
+            </joint>
+            <joint name="$(arg arm_prefix)joint1">
+                <command_interface name="position"/>
+                <state_interface name="position"/>
+                <state_interface name="velocity"/>
+            </joint>
+            <joint name="$(arg arm_prefix)joint2">
+                <command_interface name="position"/>
+                <state_interface name="position"/>
+                <state_interface name="velocity"/>
+            </joint>
+            <joint name="$(arg arm_prefix)joint3">
+                <command_interface name="position"/>
+                <state_interface name="position"/>
+                <state_interface name="velocity"/>
+            </joint>
+        </xacro:if>
+    </ros2_control>
+    <!-- Wheel friction settings -->
+    <gazebo reference="front_left_wheel_link">
+        <mu1>1.0</mu1>
+        <mu2>1.0</mu2>
+        <kp>1000000.0</kp>
+        <kd>100.0</kd>
+        <minDepth>0.001</minDepth>
+    </gazebo>
+    <gazebo reference="front_right_wheel_link">
+        <mu1>1.0</mu1>
+        <mu2>1.0</mu2>
+        <kp>1000000.0</kp>
+        <kd>100.0</kd>
+        <minDepth>0.001</minDepth>
+    </gazebo>
+    <gazebo reference="back_left_wheel_link">
+        <mu1>1.0</mu1>
+        <mu2>1.0</mu2>
+        <kp>1000000.0</kp>
+        <kd>100.0</kd>
+        <minDepth>0.001</minDepth>
+    </gazebo>
+    <gazebo reference="back_right_wheel_link">
+        <mu1>1.0</mu1>
+        <mu2>1.0</mu2>
+        <kp>1000000.0</kp>
+        <kd>100.0</kd>
+        <minDepth>0.001</minDepth>
+    </gazebo>
 </robot>

File: src/aero_description/urdf/aero.ignition.xacro (robot description, xacro)
@@ -18,30 +18,28 @@
             <gz_frame_id>lidar_link</gz_frame_id>
             <lidar>
-            <scan>
-                <horizontal>
-                    <samples>300</samples>
-                    <resolution>1.000000</resolution>
-                    <min_angle>-2.500000</min_angle>
-                    <max_angle>2.280000</max_angle>
-                </horizontal>
-            </scan>
-            <range>
-                <min>0.120000</min>
-                <max>5.5</max>
-                <resolution>0.015000</resolution>
-            </range>
-            <noise>
-                <type>gaussian</type>
-                <mean>0.0</mean>
-                <stddev>0.01</stddev>
-            </noise>
+                <scan>
+                    <horizontal>
+                        <samples>300</samples>
+                        <resolution>1.000000</resolution>
+                        <min_angle>-2.500000</min_angle>
+                        <max_angle>2.280000</max_angle>
+                    </horizontal>
+                </scan>
+                <range>
+                    <min>0.120000</min>
+                    <max>5.5</max>
+                    <resolution>0.015000</resolution>
+                </range>
+                <noise>
+                    <type>gaussian</type>
+                    <mean>0.0</mean>
+                    <stddev>0.01</stddev>
+                </noise>
             </lidar>
         </sensor>
     </gazebo>
     <gazebo>
-        <plugin filename="gz_ros2_control-system" name="gz_ros2_control::GazeboSimROS2ControlPlugin">
-            <robot_param>robot_description</robot_param>
-            <robot_param_node>robot_state_publisher</robot_param_node>
-            <parameters>$(find aero_bringup)/config/controllers.yaml</parameters>
+        <plugin filename="libgz_ros2_control-system.so" name="gz_ros2_control::GazeboSimROS2ControlPlugin">
+            <parameters>/home/ali/Desktop/Ros2_Control/install/aero_bringup/share/aero_bringup/config/controllers.yaml</parameters>
         </plugin>
         <plugin filename="libignition-gazebo-imu-system.so"

File: src/aero_description/urdf/aero.urdf.xacro (robot description, xacro)
@@ -15,11 +15,11 @@
         <xacro:include filename= "arm/arm.urdf.xacro" />
     </xacro:if>
-    <xacro:if value="$(arg use_ignition)">
+    <xacro:if value="${use_ignition}">
         <xacro:include filename="aero.ignition.xacro" />
     </xacro:if>
-    <xacro:if value="$(arg use_webots)">
+    <xacro:if value="${use_webots}">
         <xacro:include filename="aero.webots.xacro" />
     </xacro:if>
-    <xacro:if value="$(arg use_gazebo)">
+    <xacro:if value="${use_gazebo}">
         <xacro:include filename="aero.gazebo.xacro" />
     </xacro:if>

File: src/aero_description/urdf/aero_base.xacro (robot description, xacro)
@@ -253,32 +253,3 @@
         <axis xyz="0 1 0" />
     </joint>
-    <!--Ros 2 control part added -->
-    <ros2_control name="GazeboSystem" type="system">
-        <hardware>
-            <plugin>gazebo_ros2_control/GazeboSystem</plugin>
-        </hardware>
-        <joint name="left_wheel_joint">
-            <command_interface name="velocity">
-                <param name="min">-10</param>
-                <param name="max">10</param>
-            </command_interface>
-            <state_interface name="velocity"/>
-            <state_interface name="position"/>
-        </joint>
-        <joint name="right_wheel_joint">
-            <command_interface name="velocity">
-                <param name="min">-10</param>
-                <param name="max">10</param>
-            </command_interface>
-            <state_interface name="velocity"/>
-            <state_interface name="position"/>
-        </joint>
-    </ros2_control>
-    <gazebo>
-    <plugin name="gazebo_ros2_control" filename="libgazebo_ros2_control.so">
-        <!-- Use controller configs from my_robot_bringup package -->
-        <parameters>$(find my_robot_bringup)/config/my_robot_controllers.yaml</parameters>
-        <parameters>$(find my_robot_bringup)/config/ignition.yaml</parameters>
-    </plugin>
-    </gazebo>
 </robot>

File: src/aero_description/urdf/mobile_base.ros2_control.xacro (robot description, xacro)
@@ -1,32 +1,5 @@
 <?xml version="1.0"?>
 <robot xmlns:xacro="http://www.ros.org/wiki/xacro">
-    <xacro:if value="${(not use_ignition and not use_gazebo) and not use_webots}">
-        <ros2_control name="MobileBaseHardwareInterface" type="system">
-            <hardware>
-                <plugin>mock_components/GenericSystem</plugin>
-                <param name="calculate_dynamics">true</param>
-            </hardware>
-            <xacro:macro name="mock_joint" params="name">
-                <joint name="${name}">
-                    <command_interface name="velocity" />
-                    <command_interface name="position" />
-                    <state_interface name="position" />
-                    <state_interface name="velocity" />
-                </joint>
-            </xacro:macro>
-            <xacro:mock_joint name="base_back_left_wheel_joint" />
-            <xacro:mock_joint name="base_back_right_wheel_joint" />
-            <xacro:mock_joint name="base_front_left_wheel_joint" />
-            <xacro:mock_joint name="base_front_right_wheel_joint" />
-            <xacro:if value="$(arg arm_enabled)">
-                <xacro:mock_joint name="$(arg arm_prefix)joint0" />
-                <xacro:mock_joint name="$(arg arm_prefix)joint1" />
-                <xacro:mock_joint name="$(arg arm_prefix)joint2" />
-                <xacro:mock_joint name="$(arg arm_prefix)joint3" />
-                <xacro:mock_joint name="$(arg arm_prefix)joint4" />
-            </xacro:if>
-        </ros2_control>
-    </xacro:if>
-    <xacro:if value="$(arg use_ignition)">
+    <xacro:if value="${use_ignition}">
         <ros2_control name="GazeboSimSystem" type="system">
             <hardware>
@@ -45,37 +18,4 @@
             <xacro:gazebo_joint name="base_back_right_wheel_joint" />
             <xacro:gazebo_joint name="base_back_left_wheel_joint" />
-            <xacro:if value="$(arg arm_enabled)">
-                <xacro:gazebo_joint name="$(arg arm_prefix)joint0" />
-                <xacro:gazebo_joint name="$(arg arm_prefix)joint1" />
-                <xacro:gazebo_joint name="$(arg arm_prefix)joint2" />
-                <xacro:gazebo_joint name="$(arg arm_prefix)joint3" />
-                <xacro:gazebo_joint name="$(arg arm_prefix)joint4" />
-            </xacro:if>
-        </ros2_control>
-    </xacro:if>
-    <xacro:if value="${use_webots}">
-        <ros2_control name="WebotsSystem" type="system">
-            <hardware>
-                <plugin>webots_ros2_control::WebotsSystem</plugin>
-            </hardware>
-            <xacro:macro name="webots_joint" params="name">
-                <joint name="${name}">
-                    <command_interface name="velocity" />
-                    <command_interface name="position" />
-                    <state_interface name="position" />
-                    <state_interface name="velocity"/>
-                </joint>
-            </xacro:macro>
-            <xacro:webots_joint name="base_front_right_wheel_joint" />
-            <xacro:webots_joint name="base_front_left_wheel_joint" />
-            <xacro:webots_joint name="base_back_right_wheel_joint" />
-            <xacro:webots_joint name="base_back_left_wheel_joint" />
-            <xacro:if value="$(arg arm_enabled)">
-                <xacro:webots_joint name="$(arg arm_prefix)joint0" />
-                <xacro:webots_joint name="$(arg arm_prefix)joint1" />
-                <xacro:webots_joint name="$(arg arm_prefix)joint2" />
-                <xacro:webots_joint name="$(arg arm_prefix)joint3" />
-                <xacro:webots_joint name="$(arg arm_prefix)joint4" />
-            </xacro:if>
         </ros2_control>
     </xacro:if>

Commit message: final code status will be fixed

File: src/aero_description/urdf/aero.gazebo.xacro (robot description, xacro)
@@ -4,6 +4,4 @@
     <gazebo>
         <plugin filename="libgazebo_ros2_control.so" name="gazebo_ros2_control">
-            <robot_param>robot_description</robot_param>
-            <robot_param_node>robot_state_publisher</robot_param_node>
             <parameters>$(find aero_bringup)/config/controllers.yaml</parameters>
         </plugin>
@@ -14,5 +12,5 @@
             <plugin>gazebo_ros2_control/GazeboSystem</plugin>
         </hardware>
-        <!-- Wheel joints -->
+        <!-- Wheel joints - velocity controlled -->
         <joint name="base_front_left_wheel_joint">
             <command_interface name="velocity">
@@ -47,27 +45,37 @@
             <state_interface name="velocity"/>
         </joint>
-        <!-- Arm joints -->
-        <xacro:if value="$(arg arm_enabled)">
-            <joint name="$(arg arm_prefix)joint0">
-                <command_interface name="position"/>
-                <state_interface name="position"/>
-                <state_interface name="velocity"/>
-            </joint>
-            <joint name="$(arg arm_prefix)joint1">
-                <command_interface name="position"/>
-                <state_interface name="position"/>
-                <state_interface name="velocity"/>
-            </joint>
-            <joint name="$(arg arm_prefix)joint2">
-                <command_interface name="position"/>
-                <state_interface name="position"/>
-                <state_interface name="velocity"/>
-            </joint>
-            <joint name="$(arg arm_prefix)joint3">
-                <command_interface name="position"/>
-                <state_interface name="position"/>
-                <state_interface name="velocity"/>
-            </joint>
-        </xacro:if>
+        <!-- Arm joints - position controlled -->
+        <joint name="arm_joint0">
+            <command_interface name="position">
+                <param name="min">-6.28</param>
+                <param name="max">6.28</param>
+            </command_interface>
+            <state_interface name="position"/>
+            <state_interface name="velocity"/>
+        </joint>
+        <joint name="arm_joint1">
+            <command_interface name="position">
+                <param name="min">-6.28</param>
+                <param name="max">6.28</param>
+            </command_interface>
+            <state_interface name="position"/>
+            <state_interface name="velocity"/>
+        </joint>
+        <joint name="arm_joint2">
+            <command_interface name="position">
+                <param name="min">-6.28</param>
+                <param name="max">6.28</param>
+            </command_interface>
+            <state_interface name="position"/>
+            <state_interface name="velocity"/>
+        </joint>
+        <joint name="arm_joint3">
+            <command_interface name="position">
+                <param name="min">-6.28</param>
+                <param name="max">6.28</param>
+            </command_interface>
+            <state_interface name="position"/>
+            <state_interface name="velocity"/>
+        </joint>
     </ros2_control>
     <!-- Wheel friction settings -->
@@ -100,3 +108,53 @@
         <minDepth>0.001</minDepth>
     </gazebo>
+    <!-- Gazebo Classic IMU Sensor -->
+    <gazebo reference="imu_link">
+        <sensor name="imu_sensor" type="imu">
+            <always_on>true</always_on>
+            <update_rate>100</update_rate>
+            <plugin name="imu_plugin" filename="libgazebo_ros_imu_sensor.so">
+                <ros>
+                    <namespace>/</namespace>
+                    <remapping>~/out:=imu</remapping>
+                </ros>
+                <initial_orientation_as_reference>false</initial_orientation_as_reference>
+            </plugin>
+        </sensor>
+    </gazebo>
+    <!-- Gazebo Classic Lidar Sensor -->
+    <gazebo reference="lidar_link">
+        <sensor name="lidar" type="ray">
+            <always_on>true</always_on>
+            <visualize>true</visualize>
+            <update_rate>5</update_rate>
+            <ray>
+                <scan>
+                    <horizontal>
+                        <samples>300</samples>
+                        <resolution>1.0</resolution>
+                        <min_angle>-2.5</min_angle>
+                        <max_angle>2.28</max_angle>
+                    </horizontal>
+                </scan>
+                <range>
+                    <min>0.12</min>
+                    <max>5.5</max>
+                    <resolution>0.015</resolution>
+                </range>
+                <noise>
+                    <type>gaussian</type>
+                    <mean>0.0</mean>
+                    <stddev>0.01</stddev>
+                </noise>
+            </ray>
+            <plugin name="lidar_plugin" filename="libgazebo_ros_ray_sensor.so">
+                <ros>
+                    <namespace>/</namespace>
+                    <remapping>~/out:=scan</remapping>
+                </ros>
+                <output_type>sensor_msgs/LaserScan</output_type>
+                <frame_name>lidar_link</frame_name>
+            </plugin>
+        </sensor>
+    </gazebo>
 </robot>

File: src/aero_description/urdf/aero.ignition.xacro (robot description, xacro)
@@ -39,7 +39,92 @@
         </sensor>
     </gazebo>
+    <!-- ros2_control hardware interface -->
+    <ros2_control name="GazeboSystem" type="system">
+        <hardware>
+            <plugin>gz_ros2_control/GazeboSimSystem</plugin>
+        </hardware>
+        <!-- Wheel joints -->
+        <joint name="base_front_right_wheel_joint">
+            <command_interface name="velocity">
+                <param name="min">-10</param>
+                <param name="max">10</param>
+            </command_interface>
+            <state_interface name="position"/>
+            <state_interface name="velocity"/>
+        </joint>
+        <joint name="base_front_left_wheel_joint">
+            <command_interface name="velocity">
+                <param name="min">-10</param>
+                <param name="max">10</param>
+            </command_interface>
+            <state_interface name="position"/>
+            <state_interface name="velocity"/>
+        </joint>
+        <joint name="base_back_right_wheel_joint">
+            <command_interface name="velocity">
+                <param name="min">-10</param>
+                <param name="max">10</param>
+            </command_interface>
+            <state_interface name="position"/>
+            <state_interface name="velocity"/>
+        </joint>
+        <joint name="base_back_left_wheel_joint">
+            <command_interface name="velocity">
+                <param name="min">-10</param>
+                <param name="max">10</param>
+            </command_interface>
+            <state_interface name="position"/>
+            <state_interface name="velocity"/>
+        </joint>
+        <!-- Arm joints -->
+        <joint name="arm_joint0">
+            <command_interface name="position">
+                <param name="min">-3.14</param>
+                <param name="max">3.14</param>
+            </command_interface>
+            <state_interface name="position"/>
+            <state_interface name="velocity"/>
+        </joint>
+        <joint name="arm_joint1">
+            <command_interface name="position">
+                <param name="min">-3.14</param>
+                <param name="max">3.14</param>
+            </command_interface>
+            <state_interface name="position"/>
+            <state_interface name="velocity"/>
+        </joint>
+        <joint name="arm_joint2">
+            <command_interface name="position">
+                <param name="min">-3.14</param>
+                <param name="max">3.14</param>
+            </command_interface>
+            <state_interface name="position"/>
+            <state_interface name="velocity"/>
+        </joint>
+        <joint name="arm_joint3">
+            <command_interface name="position">
+                <param name="min">-3.14</param>
+                <param name="max">3.14</param>
+            </command_interface>
+            <state_interface name="position"/>
+            <state_interface name="velocity"/>
+        </joint>
+        <!-- IMU sensor -->
+        <sensor name="imu_sensor">
+            <state_interface name="orientation.x"/>
+            <state_interface name="orientation.y"/>
+            <state_interface name="orientation.z"/>
+            <state_interface name="orientation.w"/>
+            <state_interface name="angular_velocity.x"/>
+            <state_interface name="angular_velocity.y"/>
+            <state_interface name="angular_velocity.z"/>
+            <state_interface name="linear_acceleration.x"/>
+            <state_interface name="linear_acceleration.y"/>
+            <state_interface name="linear_acceleration.z"/>
+        </sensor>
+    </ros2_control>
     <gazebo>
         <plugin filename="gz_ros2_control-system" name="gz_ros2_control::GazeboSimROS2ControlPlugin">
-            <parameters>/home/ali/Desktop/Ros2_Control/install/aero_bringup/share/aero_bringup/config/controllers.yaml</parameters>
+            <parameters>$(find aero_bringup)/config/controllers.yaml</parameters>
             <robot_param>robot_description</robot_param>
             <robot_param_node>robot_state_publisher</robot_param_node>
